Commit message: Reskin Bravo URDF with realistic materials and grouped deck colors

File: pybravo/model/pybravo_urdf/robot.urdf (robot description, URDF)
Before this commit: robot robot, 43 links, 42 joints
Links:
- link 384_head_384_head: geometry collision mesh filename=package://assets/384_head.stl; visual mesh filename=package://assets/bravo_head_barrels.stl
- link xgantry_xgantry: geometry collision mesh filename=package://assets/xgantry.stl; visual mesh filename=package://assets/bravo_brand_emblem.stl
- link ygantry_ygantry: geometry collision mesh filename=package://assets/ygantry.stl; visual mesh filename=package://assets/bravo_carriage_cover.stl

Commit message: Align gripper grasp geometry and restore real liquid well depth

File: pybravo/model/pybravo_urdf/robot.urdf (robot description, URDF)
Before this commit: robot robot, 43 links, 42 joints
Joints:
- joint zaxis-gripper: origin xyz=0.100478 -0.224926 -0.0530846 rpy=1.5708 8.63559e-42 -5.71589e-35 -> xyz=0.078228 -0.224926 -0.0530846 rpy=1.5708 8.63559e-42 -5.71589e-35
